File: hardware/ecp5-i5/spice/kicad/t1_frontend.kicad_sch (KiCad schematic)
At the start: 32 parts, among them Q1 BS250, Q2 BS250, Q3 2N7000, Q4 2N7000, Q5 2N3904, Q6 2N3904, Q7 2N7000, Q8 2N3904, Q9 2N7002, U3 OPA171

Commit message: feat(hardware): 完整 tVNS 前端原理图(逻辑+桥+sink+安全层+接口) + BOM
51 器件/71 unit 实例/38 网，kicad-cli netlist 校验全通。生成器支持多单元符号(74HC0x/LM393)。含 BOM(含封装/耐压/精度)。
Parts:
- added C3, C4, C5, C6, C7, C8: 100n, symbol Device:C
- added J1: CTRL, symbol Connector_Generic:Conn_01x08
- added J2: ELECTRODE, symbol Connector_Generic:Conn_01x02
- added R16, R19, R20: 10k, symbol Device:R
- added R17: 39k, symbol Device:R
- added R18: 1k, symbol Device:R
- added U1: SN74HC04, symbol 74xx:74HC04
- added U2, U6: SN74HC08, symbol 74xx:74LS08
- added U4: LM393, symbol Comparator:LM393
- added U5: SN74HC00, symbol 74xx:74HC00
- added U7: TL431, symbol Reference_Voltage:TL431LP
Connections:
- net A1: now also U2.8
- net A2: now also U2.11
- net EL1: now also J2.1 (Pin_1)
- net ENB: now also U1.6
- net GND: now also C3.2, C4.2, C5.2, C6.2, C7.2, C8.2, J1.4 (Pin_4), R18.2, U1.11, U1.13, U1.7 (GND), U1.9, U2.7 (GND), U4.4 (V-), U4.5 (+), U4.6 (-), U5.10, U5.12, U5.13, U5.7 (GND), U5.9, U6.10, U6.12, U6.13, U6.4, U6.5, U6.7 (GND), U6.9, U7.2 (A); no longer RV1.1
- net MID2: now also J2.2 (Pin_2)
- net S: now also U4.3 (+)
- net VS: now also J1.1 (Pin_1)
- net V12 renamed +12V
- net +12V: now also C8.1, J1.2 (Pin_2)
- net V5 renamed VDDA
- new net +5V: C3.1, C4.1, C5.1, C6.1, C7.1, J1.3 (Pin_3), R16.1, R19.1, R20.1, RV1.1, U1.14 (VCC), U2.14 (VCC), U4.8 (V+), U5.14 (VCC), U6.14 (VCC)
- new net EN_MCU: J1.7 (Pin_7), U6.1
- new net EN_OUT: U1.5, U2.1, U2.4, U6.3
- new net EN_SAFE: U5.3, U5.4, U6.2
- new net IN1: J1.5 (Pin_5), U1.1, U2.2
- new net IN1B: U1.2, U2.13
- new net IN2: J1.6 (Pin_6), U1.3, U2.5
- new net IN2B: U1.4, U2.10
- new net N1: U2.3, U2.9
- new net N2: U2.12, U2.6
- new net QLB: U5.2, U5.6
- new net TL_K: R17.1, R19.2, U7.1 (REF), U7.3 (K)
- new net TRIP_CMP: R16.2, U4.1, U5.1
- new net TRIP_RST: J1.8 (Pin_8), R20.2, U5.5
- new net VREF60: R17.2, R18.1, U4.2 (-)

Commit message: feat(hardware): KiCad 工程(.kicad_pro/.kicad_pcb) + 器件封装分配
补工程文件(可用 KiCad 打开工程)；为全部器件分配 Footprint(SMD优先)，供 GUI 'Update PCB from Schematic' 一键落板。忽略 .history/__pycache__/*.lck。
Parts:
- C1, C3, C4, C5, C6, C7, C8: footprint (none) -> Capacitor_SMD:C_0603_1608Metric
- C2: footprint (none) -> Capacitor_THT:C_Rect_L7.0mm_W2.5mm_P5.00mm
- D1, D2: footprint (none) -> Diode_SMD:D_SOD-123
- D3, D4: footprint (none) -> Diode_SMD:D_SMA
- J1: footprint (none) -> Connector_PinHeader_2.54mm:PinHeader_1x08_P2.54mm_Vertical
- J2: footprint (none) -> TerminalBlock:TerminalBlock_bornier-2_P5.08mm
- Q1, Q2, Q3, Q4, Q5, Q6, Q7, Q8: footprint (none) -> Package_TO_SOT_THT:TO-92_Inline
- Q9, U7: footprint (none) -> Package_TO_SOT_SMD:SOT-23
- R1, R10, R11, R12, R13, R14, R15, R16, R17, R18, R19, R2, R20, R3, R4, R5, R6, R7, R8: footprint (none) -> Resistor_SMD:R_0805_2012Metric
- R9: footprint (none) -> Resistor_SMD:R_1206_3216Metric
- RV1: footprint (none) -> Potentiometer_THT:Potentiometer_Bourns_3296W_Vertical
- U1, U2, U5, U6: footprint (none) -> Package_DIP:DIP-14_W7.62mm
- U3: footprint (none) -> Package_TO_SOT_SMD:SOT-23-5
- U4: footprint (none) -> Package_SO:SOIC-8_3.9x4.9mm_P1.27mm

Commit message: fix(hardware): 修正 J2 封装为 TerminalBlock_MaiXu_MX126-5.0-02P (原 bornier 名不存在)
Parts:
- J2: footprint TerminalBlock:TerminalBlock_bornier-2_P5.08mm -> TerminalBlock:TerminalBlock_MaiXu_MX126-5.0-02P_1x02_P5.00mm
Changed lines of the file:
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@@
 		(property "Reference" "J2" (at 360 297.5 0) (effects (font (size 1.27 1.27)) (hide yes)))
 		(property "Value" "ELECTRODE" (at 360 302.5 0) (effects (font (size 1.27 1.27)) (hide yes)))
-		(property "Footprint" "TerminalBlock:TerminalBlock_bornier-2_P5.08mm" (at 360 300 0) (effects (font (size 1.27 1.27)) (hide yes)))
+		(property "Footprint" "TerminalBlock:TerminalBlock_MaiXu_MX126-5.0-02P_1x02_P5.00mm" (at 360 300 0) (effects (font (size 1.27 1.27)) (hide yes)))
 		(property "Datasheet" "~" (at 360 300 0) (effects (font (size 1.27 1.27)) (hide yes)))
 		(instances (project "feelings" (path "/00000000-0000-0000-0000-000000000001" (reference "J2") (unit 1))))
