File: hardware/ecp5-i5/spice/kicad/t1_frontend.kicad_sch (KiCad schematic)
At the start: 51 parts, among them J1 CTRL, J2 ELECTRODE, Q1 BS250, Q2 BS250, Q3 2N7000, Q4 2N7000, Q5 2N3904, Q6 2N3904, Q7 2N7000, Q8 2N3904, Q9 2N7002, U1 SN74HC04, U2 SN74HC08, U3 OPA171, U4 LM393, U5 SN74HC00, U6 SN74HC08, U7 TL431

Commit message: feat(hardware): LS 栅阻(22Ω)+下拉、QS 栅阻 1k→100Ω、界面电压采样(分压+AMC1351+J3)
Q3/Q4 加 22Ω 栅阻 + 10k 下拉(抑振铃/失效态 OFF)；QS 栅阻 1k→100Ω(提速)；新增界面电压采样：R25/R26 分压 → 隔离放大器 U8(AMC1351) → J3 送采集侧。netlist 43 网全通。
Parts:
- added C3, C4, C5, C6, C7, C8: 100n, Capacitor_SMD:C_0603_1608Metric, symbol Device:C
- added J1: CTRL, Connector_PinHeader_2.54mm:PinHeader_1x08_P2.54mm_Vertical, symbol Connector_Generic:Conn_01x08
- added J2: ELECTRODE, TerminalBlock:TerminalBlock_MaiXu_MX126-5.0-02P_1x02_P5.00mm, symbol Connector_Generic:Conn_01x02
- J3: renamed from U2; value SN74HC08 -> VZ_OUT; footprint Package_DIP:DIP-14_W7.62mm -> Connector_PinHeader_2.54mm:PinHeader_1x03_P2.54mm_Vertical; symbol 74xx:74LS08 -> Connector_Generic:Conn_01x03
- R16: renamed from C4; value 100n -> 10k; footprint Capacitor_SMD:C_0603_1608Metric -> Resistor_SMD:R_0805_2012Metric; symbol Device:C -> Device:R
- R17: renamed from C5; value 100n -> 39k; footprint Capacitor_SMD:C_0603_1608Metric -> Resistor_SMD:R_0805_2012Metric; symbol Device:C -> Device:R
- R18: renamed from C6; value 100n -> 1k; footprint Capacitor_SMD:C_0603_1608Metric -> Resistor_SMD:R_0805_2012Metric; symbol Device:C -> Device:R
- R19: renamed from C7; value 100n -> 10k; footprint Capacitor_SMD:C_0603_1608Metric -> Resistor_SMD:R_0805_2012Metric; symbol Device:C -> Device:R
- R20: renamed from C8; value 100n -> 10k; footprint Capacitor_SMD:C_0603_1608Metric -> Resistor_SMD:R_0805_2012Metric; symbol Device:C -> Device:R
- R21, R22: renamed from U1; value SN74HC04 -> 22R; footprint Package_DIP:DIP-14_W7.62mm -> Resistor_SMD:R_0805_2012Metric; symbol 74xx:74HC04 -> Device:R
- R23, R24: renamed from U1; value SN74HC04 -> 10k; footprint Package_DIP:DIP-14_W7.62mm -> Resistor_SMD:R_0805_2012Metric; symbol 74xx:74HC04 -> Device:R
- R25: renamed from U1; value SN74HC04 -> 1M; footprint Package_DIP:DIP-14_W7.62mm -> Resistor_SMD:R_0805_2012Metric; symbol 74xx:74HC04 -> Device:R
- R26: renamed from U1; value SN74HC04 -> 51k; footprint Package_DIP:DIP-14_W7.62mm -> Resistor_SMD:R_0805_2012Metric; symbol 74xx:74HC04 -> Device:R
- R7: value 1k -> 100R
- U1: renamed from U2; value SN74HC08 -> SN74HC04; symbol 74xx:74LS08 -> 74xx:74HC04
- U1: renamed from U4; value LM393 -> SN74HC04; footprint Package_SO:SOIC-8_3.9x4.9mm_P1.27mm -> Package_DIP:DIP-14_W7.62mm; symbol Comparator:LM393 -> 74xx:74HC04
- U2: renamed from U5; value SN74HC00 -> SN74HC08; symbol 74xx:74HC00 -> 74xx:74LS08
- U4: renamed from U6; value SN74HC08 -> LM393; footprint Package_DIP:DIP-14_W7.62mm -> Package_SO:SOIC-8_3.9x4.9mm_P1.27mm; symbol 74xx:74LS08 -> Comparator:LM393
- U5: renamed from U6; value SN74HC08 -> SN74HC00; symbol 74xx:74LS08 -> 74xx:74HC00
- U5: renamed from U7; value TL431 -> SN74HC00; footprint Package_TO_SOT_SMD:SOT-23 -> Package_DIP:DIP-14_W7.62mm; symbol Reference_Voltage:TL431LP -> 74xx:74HC00
- U5: renamed from R16; value 10k -> SN74HC00; footprint Resistor_SMD:R_0805_2012Metric -> Package_DIP:DIP-14_W7.62mm; symbol Device:R -> 74xx:74HC00
- U5: renamed from R17; value 39k -> SN74HC00; footprint Resistor_SMD:R_0805_2012Metric -> Package_DIP:DIP-14_W7.62mm; symbol Device:R -> 74xx:74HC00
- U6: renamed from R18; value 1k -> SN74HC08; footprint Resistor_SMD:R_0805_2012Metric -> Package_DIP:DIP-14_W7.62mm; symbol Device:R -> 74xx:74LS08
- U6: renamed from R19; value 10k -> SN74HC08; footprint Resistor_SMD:R_0805_2012Metric -> Package_DIP:DIP-14_W7.62mm; symbol Device:R -> 74xx:74LS08
- U6: renamed from R20; value 10k -> SN74HC08; footprint Resistor_SMD:R_0805_2012Metric -> Package_DIP:DIP-14_W7.62mm; symbol Device:R -> 74xx:74LS08
- U6: renamed from J1; value CTRL -> SN74HC08; footprint Connector_PinHeader_2.54mm:PinHeader_1x08_P2.54mm_Vertical -> Package_DIP:DIP-14_W7.62mm; symbol Connector_Generic:Conn_01x08 -> 74xx:74LS08
- U6: renamed from J2; value ELECTRODE -> SN74HC08; footprint TerminalBlock:TerminalBlock_MaiXu_MX126-5.0-02P_1x02_P5.00mm -> Package_DIP:DIP-14_W7.62mm; symbol Connector_Generic:Conn_01x02 -> 74xx:74LS08
- U7: renamed from C3; value 100n -> TL431; footprint Capacitor_SMD:C_0603_1608Metric -> Package_TO_SOT_SMD:SOT-23; symbol Device:C -> Reference_Voltage:TL431LP
- U8: renamed from U1; value SN74HC04 -> AMC1351; footprint Package_DIP:DIP-14_W7.62mm -> Package_SO:SOIC-8_7.5x5.85mm_P1.27mm; symbol 74xx:74HC04 -> Isolator_Analog:AMC1351DWV
Connections:
- net +12V: now also C8.1, J1.2 (Pin_2); no longer R20.1, U6.2 (Pin_2)
- net +5V: now also R20.1, U1.14 (VCC), U4.8 (V+), U5.14 (VCC), U6.14 (VCC), U8.1 (VDD1), C3.1, C4.1, C5.1, C6.1, C7.1, J1.3 (Pin_3); no longer R17.1, R18.1, U1.14 (VCC), U1.8 (V+), U5.1, U5.14 (VCC), U6.1, U6.1, U6.3 (Pin_3), U7.1, U8.14 (VCC)
- net A1: now also R21.1, U2.8; no longer Q4.2 (G), U1.8
- net A2: now also R22.1, U2.11; no longer Q3.2 (G), U1.11
- net EL1: now also R25.1, J2.1 (Pin_1); no longer U6.1 (Pin_1)
- net ENB: now also U1.6; no longer R23.6
- net EN_MCU: now also U6.1, J1.7 (Pin_7); no longer U4.1, U6.7 (Pin_7)
- net EN_OUT: now also U1.5, U2.1, U2.4, U6.3; no longer J3.1, R23.5, U1.4, U4.3
- net EN_SAFE: now also U5.3, U5.4, U6.2; no longer U2.3, U2.4, U4.2
- net GND: now also J3.3 (Pin_3), R23.2, R24.2, U1.11, U1.13, U1.7 (GND), U1.9, U4.4 (V-), U4.6 (-), U5.10, U5.12, U5.13, U5.7 (GND), U5.9, U6.10, U6.12, U6.13, U6.4, U6.5, U6.7 (GND), U6.9, U8.5 (GND2), C3.2, C4.2, C5.2, C6.2, C7.2, C8.2, J1.4 (Pin_4); no longer R16.2, R17.2, R19.2, R20.2, R24.9, R25.11, R26.13, U1.4 (V-), U1.5 (+), U1.6 (-), U1.7 (GND), U2.10, U2.12, U2.13, U2.9, U4.10, U4.4, U4.9, U5.12, U5.13, U5.2 (A), U5.7 (GND), U6.2, U6.4 (Pin_4), U8.7 (GND)
- net IN1: now also U1.1, U2.2, J1.5 (Pin_5); no longer J3.2, R21.1, U6.5 (Pin_5)
- net IN1B: now also U1.2, U2.13; no longer R21.2, U1.13
- net IN2: now also U1.3, U2.5, J1.6 (Pin_6); no longer R22.3, U1.5, U6.6 (Pin_6)
- net IN2B: now also U1.4, U2.10; no longer R22.4, U1.10
- net MID2: now also R26.2, U8.3 (GND1), U8.4 (GND1), J2.2 (Pin_2); no longer U6.2 (Pin_2)
- net N1: now also U2.3, U2.9; no longer J3.3, U1.9
- net N2: now also U2.12, U2.6; no longer U1.12, U1.6
- net QLB: now also U5.2, U5.6; no longer U2.2, U2.6
- net S: now also U4.3 (+); no longer U1.3 (+)
- net TL_K: now also R17.1, R19.2, U7.1 (REF), U7.3 (K); no longer U5.1, U5.1 (REF), U5.3 (K), U6.2
- net TRIP_CMP: now also R16.2, U4.1, U5.1; no longer U1.1, U2.1, U5.2
- net TRIP_RST: now also R20.2, U5.5, J1.8 (Pin_8); no longer U2.5, U6.2, U6.8 (Pin_8)
- net VDDA: now also U8.8 (VDD2)
- net VREF60: now also R17.2, R18.1, U4.2 (-); no longer U1.2 (-), U5.2, U6.1
- net VS: now also J1.1 (Pin_1); no longer U6.1 (Pin_1)
- new net ISO_N: J3.2 (Pin_2), U8.6 (OUTN)
- new net ISO_P: J3.1 (Pin_1), U8.7 (OUTP)
- new net LG1: Q3.2 (G), R22.2, R23.1
- new net LG2: Q4.2 (G), R21.2, R24.1
- new net VZ: R25.2, R26.1, U8.2 (IN)
Changed lines of the file:
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@@
 		(exclude_from_sim no) (in_bom yes) (on_board yes) (dnp no)
 		(property "Reference" "R7" (at 480 127.5 0) (effects (font (size 1.27 1.27)) (hide yes)))
-		(property "Value" "1k" (at 480 132.5 0) (effects (font (size 1.27 1.27)) (hide yes)))
+		(property "Value" "100R" (at 480 132.5 0) (effects (font (size 1.27 1.27)) (hide yes)))
 		(property "Footprint" "Resistor_SMD:R_0805_2012Metric" (at 480 130 0) (effects (font (size 1.27 1.27)) (hide yes)))
 		(property "Datasheet" "~" (at 480 130 0) (effects (font (size 1.27 1.27)) (hide yes)))
@@
 	)
 	(symbol
+		(lib_id "Device:R")
+		(at 280 180 0)
+		(unit 1)
+		(exclude_from_sim no) (in_bom yes) (on_board yes) (dnp no)
+		(property "Reference" "R21" (at 280 177.5 0) (effects (font (size 1.27 1.27)) (hide yes)))
+		(property "Value" "22R" (at 280 182.5 0) (effects (font (size 1.27 1.27)) (hide yes)))
+		(property "Footprint" "Resistor_SMD:R_0805_2012Metric" (at 280 180 0) (effects (font (size 1.27 1.27)) (hide yes)))
+		(property "Datasheet" "~" (at 280 180 0) (effects (font (size 1.27 1.27)) (hide yes)))
+		(instances (project "feelings" (path "/00000000-0000-0000-0000-000000000001" (reference "R21") (unit 1))))
+	)
+	(symbol
+		(lib_id "Device:R")
+		(at 130 230 0)
+		(unit 1)
+		(exclude_from_sim no) (in_bom yes) (on_board yes) (dnp no)
+		(property "Reference" "R22" (at 130 227.5 0) (effects (font (size 1.27 1.27)) (hide yes)))
+		(property "Value" "22R" (at 130 232.5 0) (effects (font (size 1.27 1.27)) (hide yes)))
+		(property "Footprint" "Resistor_SMD:R_0805_2012Metric" (at 130 230 0) (effects (font (size 1.27 1.27)) (hide yes)))
+		(property "Datasheet" "~" (at 130 230 0) (effects (font (size 1.27 1.27)) (hide yes)))
+		(instances (project "feelings" (path "/00000000-0000-0000-0000-000000000001" (reference "R22") (unit 1))))
+	)
+	(symbol
+		(lib_id "Device:R")
+		(at 80 230 0)
+		(unit 1)
+		(exclude_from_sim no) (in_bom yes) (on_board yes) (dnp no)
+		(property "Reference" "R23" (at 80 227.5 0) (effects (font (size 1.27 1.27)) (hide yes)))
+		(property "Value" "10k" (at 80 232.5 0) (effects (font (size 1.27 1.27)) (hide yes)))
+		(property "Footprint" "Resistor_SMD:R_0805_2012Metric" (at 80 230 0) (effects (font (size 1.27 1.27)) (hide yes)))
+		(property "Datasheet" "~" (at 80 230 0) (effects (font (size 1.27 1.27)) (hide yes)))
+		(instances (project "feelings" (path "/00000000-0000-0000-0000-000000000001" (reference "R23") (unit 1))))
+	)
+	(symbol
+		(lib_id "Device:R")
+		(at 180 230 0)
+		(unit 1)
+		(exclude_from_sim no) (in_bom yes) (on_board yes) (dnp no)
+		(property "Reference" "R24" (at 180 227.5 0) (effects (font (size 1.27 1.27)) (hide yes)))
+		(property "Value" "10k" (at 180 232.5 0) (effects (font (size 1.27 1.27)) (hide yes)))
+		(property "Footprint" "Resistor_SMD:R_0805_2012Metric" (at 180 230 0) (effects (font (size 1.27 1.27)) (hide yes)))
+		(property "Datasheet" "~" (at 180 230 0) (effects (font (size 1.27 1.27)) (hide yes)))
+		(instances (project "feelings" (path "/00000000-0000-0000-0000-000000000001" (reference "R24") (unit 1))))
+	)
+	(symbol
+		(lib_id "Device:R")
+		(at 530 400 0)
+		(unit 1)
+		(exclude_from_sim no) (in_bom yes) (on_board yes) (dnp no)
+		(property "Reference" "R25" (at 530 397.5 0) (effects (font (size 1.27 1.27)) (hide yes)))
+		(property "Value" "1M" (at 530 402.5 0) (effects (font (size 1.27 1.27)) (hide yes)))
+		(property "Footprint" "Resistor_SMD:R_0805_2012Metric" (at 530 400 0) (effects (font (size 1.27 1.27)) (hide yes)))
+		(property "Datasheet" "~" (at 530 400 0) (effects (font (size 1.27 1.27)) (hide yes)))
+		(instances (project "feelings" (path "/00000000-0000-0000-0000-000000000001" (reference "R25") (unit 1))))
+	)
+	(symbol
+		(lib_id "Device:R")
+		(at 580 400 0)
+		(unit 1)
+		(exclude_from_sim no) (in_bom yes) (on_board yes) (dnp no)
+		(property "Reference" "R26" (at 580 397.5 0) (effects (font (size 1.27 1.27)) (hide yes)))
+		(property "Value" "51k" (at 580 402.5 0) (effects (font (size 1.27 1.27)) (hide yes)))
+		(property "Footprint" "Resistor_SMD:R_0805_2012Metric" (at 580 400 0) (effects (font (size 1.27 1.27)) (hide yes)))
+		(property "Datasheet" "~" (at 580 400 0) (effects (font (size 1.27 1.27)) (hide yes)))
+		(instances (project "feelings" (path "/00000000-0000-0000-0000-000000000001" (reference "R26") (unit 1))))
+	)
+	(symbol
+		(lib_id "Isolator_Analog:AMC1351DWV")
+		(at 480 400 0)
+		(unit 1)
+		(exclude_from_sim no) (in_bom yes) (on_board yes) (dnp no)
+		(property "Reference" "U8" (at 480 397.5 0) (effects (font (size 1.27 1.27)) (hide yes)))
+		(property "Value" "AMC1351" (at 480 402.5 0) (effects (font (size 1.27 1.27)) (hide yes)))
+		(property "Footprint" "Package_SO:SOIC-8_7.5x5.85mm_P1.27mm" (at 480 400 0) (effects (font (size 1.27 1.27)) (hide yes)))
+		(property "Datasheet" "~" (at 480 400 0) (effects (font (size 1.27 1.27)) (hide yes)))
+		(instances (project "feelings" (path "/00000000-0000-0000-0000-000000000001" (reference "U8") (unit 1))))
+	)
+	(symbol
+		(lib_id "Connector_Generic:Conn_01x03")
+		(at 1250 80 0)
+		(unit 1)
+		(exclude_from_sim no) (in_bom yes) (on_board yes) (dnp no)
+		(property "Reference" "J3" (at 1250 77.5 0) (effects (font (size 1.27 1.27)) (hide yes)))
+		(property "Value" "VZ_OUT" (at 1250 82.5 0) (effects (font (size 1.27 1.27)) (hide yes)))
+		(property "Footprint" "Connector_PinHeader_2.54mm:PinHeader_1x03_P2.54mm_Vertical" (at 1250 80 0) (effects (font (size 1.27 1.27)) (hide yes)))
+		(property "Datasheet" "~" (at 1250 80 0) (effects (font (size 1.27 1.27)) (hide yes)))
+		(instances (project "feelings" (path "/00000000-0000-0000-0000-000000000001" (reference "J3") (unit 1))))
+	)
+	(symbol
 		(lib_id "74xx:74HC04")
 		(at 880 130 0)
@@
 		(effects (font (size 1.0 1.0)) (justify left bottom))
 	)
+	(label "GND"
+		(at 80.0 233.81 0)
+		(effects (font (size 1.0 1.0)) (justify left bottom))
+	)
+	(label "GND"
+		(at 180.0 233.81 0)
+		(effects (font (size 1.0 1.0)) (justify left bottom))
+	)
+	(label "GND"
+		(at 482.54 410.16 0)
+		(effects (font (size 1.0 1.0)) (justify left bottom))
+	)
+	(label "GND"
+		(at 1244.92 82.54 0)
+		(effects (font (size 1.0 1.0)) (justify left bottom))
+	)
 	(label "+12V"
 		(at 477.46 87.62 0)
@@
 		(effects (font (size 1.0 1.0)) (justify left bottom))
 	)
+	(label "+5V"
+		(at 477.46 389.84 0)
+		(effects (font (size 1.0 1.0)) (justify left bottom))
+	)
 	(label "VDDA"
 		(at 580.0 126.19 0)
 		(effects (font (size 1.0 1.0)) (justify left bottom))
 	)
+	(label "VDDA"
+		(at 482.54 389.84 0)
+		(effects (font (size 1.0 1.0)) (justify left bottom))
+	)
 	(label "A1"
 		(at 987.62 180.0 0)
@@
 	)
 	(label "A1"
-		(at 74.92 130.0 0)
+		(at 130.0 126.19 0)
 		(effects (font (size 1.0 1.0)) (justify left bottom))
 	)
 	(label "A1"
-		(at 130.0 126.19 0)
+		(at 280.0 176.19 0)
 		(effects (font (size 1.0 1.0)) (justify left bottom))
 	)
@@
 	)
 	(label "A2"
+		(at 80.0 176.19 0)
+		(effects (font (size 1.0 1.0)) (justify left bottom))
+	)
+	(label "A2"
+		(at 130.0 226.19 0)
+		(effects (font (size 1.0 1.0)) (justify left bottom))
+	)
+	(label "LG1"
+		(at 130.0 233.81 0)
+		(effects (font (size 1.0 1.0)) (justify left bottom))
+	)
+	(label "LG1"
 		(at 174.92 80.0 0)
 		(effects (font (size 1.0 1.0)) (justify left bottom))
 	)
-	(label "A2"
-		(at 80.0 176.19 0)
+	(label "LG1"
+		(at 80.0 226.19 0)
+		(effects (font (size 1.0 1.0)) (justify left bottom))
+	)
+	(label "LG2"
+		(at 280.0 183.81 0)
+		(effects (font (size 1.0 1.0)) (justify left bottom))
+	)
+	(label "LG2"
+		(at 74.92 130.0 0)
+		(effects (font (size 1.0 1.0)) (justify left bottom))
+	)
+	(label "LG2"
+		(at 180.0 226.19 0)
 		(effects (font (size 1.0 1.0)) (justify left bottom))
 	)
@@
 		(effects (font (size 1.0 1.0)) (justify left bottom))
 	)
+	(label "MID2"
+		(at 580.0 403.81 0)
+		(effects (font (size 1.0 1.0)) (justify left bottom))
+	)
+	(label "MID2"
+		(at 477.46 410.16 0)
+		(effects (font (size 1.0 1.0)) (justify left bottom))
+	)
+	(label "MID2"
+		(at 477.46 410.16 0)
+		(effects (font (size 1.0 1.0)) (justify left bottom))
+	)
 	(label "B"
 		(at 182.54 85.08 0)
@@
 		(effects (font (size 1.0 1.0)) (justify left bottom))
 	)
+	(label "EL1"
+		(at 530.0 396.19 0)
+		(effects (font (size 1.0 1.0)) (justify left bottom))
+	)
 	(label "AWD"
 		(at 580.0 133.81 0)
@@
 		(effects (font (size 1.0 1.0)) (justify left bottom))
 	)
+	(label "VZ"
+		(at 530.0 403.81 0)
+		(effects (font (size 1.0 1.0)) (justify left bottom))
+	)
+	(label "VZ"
+		(at 580.0 396.19 0)
+		(effects (font (size 1.0 1.0)) (justify left bottom))
+	)
+	(label "VZ"
+		(at 469.84 400.0 0)
+		(effects (font (size 1.0 1.0)) (justify left bottom))
+	)
+	(label "ISO_P"
+		(at 490.16 397.46 0)
+		(effects (font (size 1.0 1.0)) (justify left bottom))
+	)
+	(label "ISO_P"
+		(at 1244.92 77.46 0)
+		(effects (font (size 1.0 1.0)) (justify left bottom))
+	)
+	(label "ISO_N"
+		(at 490.16 402.54 0)
+		(effects (font (size 1.0 1.0)) (justify left bottom))
+	)
+	(label "ISO_N"
+		(at 1244.92 80.0 0)
+		(effects (font (size 1.0 1.0)) (justify left bottom))
+	)
